File: Logic_Probe.sch (EAGLE design)
At the start: 26 parts, among them IC1 NE555N, IC2 QUAD_OPAMPP, Q1 MOSFET-NCH-2N7002PW, Q2 MOSFET-NCH-2N7002PW, Q3 MOSFET-NCH-2N7002PW

Commit message: Final Schematic
Parts:
- added FRAME1: FRAME-LETTER, SparkFun-Aesthetics:FRAME-LETTER
Other:
- moved on the sheet: C1, D2, D3, IC1, IC2A, IC2B, IC2C, IC2D, LED1, LED2, LED3, Q1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
